Commit message: add kuka reaching task (not working)

File: src/stage/envs/urdf/kuka/iiwa14.urdf (robot description, URDF)
Before this commit: robot KUKAiiwa14, 8 links, 7 joints
Links:
- link iiwaBase: mass None -> 0.0
Joints:
- joint A1: limit effort=30 velocity=1.0 -> lower=-2.96705972839 upper=2.96705972839 effort=30 velocity=1.0
- joint A2: limit effort=30 velocity=1.0 -> lower=-2.09439510239 upper=2.09439510239 effort=30 velocity=1.0
- joint A3: limit effort=30 velocity=1.0 -> lower=-2.96705972839 upper=2.96705972839 effort=30 velocity=1.0
- joint A4: limit effort=30 velocity=1.0 -> lower=-2.09439510239 upper=2.09439510239 effort=30 velocity=1.0
- joint A5: limit effort=30 velocity=1.0 -> lower=-2.96705972839 upper=2.96705972839 effort=30 velocity=1.0
- joint A6: limit effort=30 velocity=1.0 -> lower=-2.09439510239 upper=2.09439510239 effort=30 velocity=1.0
- joint A7: limit effort=30 velocity=1.0 -> lower=-3.05432619099 upper=3.05432619099 effort=30 velocity=1.0
